Commit message: moved stl and changed urdf bindings

File: ros2_workspace/src/simplebot_description/src/description/simplebot_description.urdf (robot description, URDF)
Before this commit: robot onshape, 6 links, 5 joints
Links:
- link frame2: geometry collision mesh filename=file://$(find simplebot_description)/meshes/frame2.stl; visual mesh filename=file://$(find simplebot_description)/meshes/frame2.stl
- link front_left: geometry collision mesh filename=file://$(find simplebot_description)/meshes/front_left.stl; visual mesh filename=file://$(find simplebot_description)/meshes/front_left.stl
- link front_right: geometry collision mesh filename=file://$(find simplebot_description)/meshes/front_right.stl; visual mesh filename=file://$(find simplebot_description)/meshes/front_right.stl
- link rear_left: geometry collision mesh filename=file://$(find simplebot_description)/meshes/rear_left.stl; visual mesh filename=file://$(find simplebot_description)/meshes/rear_left.stl
- link rear_right: geometry collision mesh filename=file://$(find simplebot_description)/meshes/rear_right.stl; visual mesh filename=file://$(find simplebot_description)/meshes/rear_right.stl
