Commit message: urdf + simplebot_description

File: onshape/simplebot2/robot.urdf (robot description, URDF)
Before this commit: robot simplebot2, 5 links, 4 joints
Links:
- removed link base_link
- added link bottom_bracket, mass 0.426296; collision mesh filename=package://assets/bottom_bracket.stl; collision mesh filename=package://assets/frame1.stl
- link part_1: geometry collision mesh filename=package://assets/part_1__3.stl; visual mesh filename=package://assets/part_1__3.stl
- link part_1_2: geometry collision mesh filename=package://assets/part_1__3.stl; visual mesh filename=package://assets/part_1__3.stl
- link part_1_3: geometry collision mesh filename=package://assets/part_1__3.stl; visual mesh filename=package://assets/part_1__3.stl
- link part_1_4: geometry collision mesh filename=package://assets/part_1__3.stl; visual mesh filename=package://assets/part_1__3.stl
Joints:
- joint Revolute 1: parent base_link -> bottom_bracket; type continuous -> revolute
- joint Revolute 2: parent base_link -> bottom_bracket; type continuous -> revolute
- joint Revolute 3: parent base_link -> bottom_bracket; type continuous -> revolute
- joint Revolute 4: parent base_link -> bottom_bracket; type continuous -> revolute

File: ros2_workspace/src/simplebot_description/src/description/old/simplebot_description.urdf (robot description, URDF)
Before this commit: robot simplebot2, 5 links, 4 joints
Links:
- removed link base_link
- added link bottom_bracket, mass 0.426296; collision mesh filename=file://$(find simplebot_description)/meshes/bottom_bracket.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; collision mesh filename=file://$(find simplebot_description)/meshes/frame1.stl
Joints:
- joint Revolute 1: parent base_link -> bottom_bracket; type continuous -> revolute
- joint Revolute 2: parent base_link -> bottom_bracket; type continuous -> revolute
- joint Revolute 3: parent base_link -> bottom_bracket; type continuous -> revolute
- joint Revolute 4: parent base_link -> bottom_bracket; type continuous -> revolute

File: ros2_workspace/src/simplebot_description/src/description/robot.urdf (robot description, URDF)
Before this commit: robot simplebot2, 5 links, 4 joints
Joints:
- joint Revolute 1: type continuous -> revolute
- joint Revolute 2: type continuous -> revolute
- joint Revolute 3: origin xyz=-0.0629675 0.253869 -0.0793943 rpy=-1.5708 -0 1.5708 -> xyz=-0.0629675 0.253869 -0.0793943 rpy=1.5708 -0 1.5708; type continuous -> revolute
- joint Revolute 4: origin xyz=-0.0629675 0.123869 -0.0793943 rpy=-1.5708 -0 1.5708 -> xyz=-0.0629675 0.123869 -0.0793943 rpy=1.5708 -0 1.5708; type continuous -> revolute

Commit message: description works

File: onshape/simplebot2/robot.urdf (robot description, URDF)
Before this commit: robot simplebot2, 5 links, 4 joints
Joints:
- joint Revolute 1: origin xyz=0.143049 0.123869 -0.0793943 rpy=-1.5708 -0 1.5708 -> xyz=-0.065 -0.103008 0.0125 rpy=-1.5708 -0 -1.66533e-16
- joint Revolute 2: origin xyz=0.143049 0.253869 -0.0793943 rpy=-1.5708 -0 1.5708 -> xyz=0.065 -0.103008 0.0125 rpy=-1.5708 -0 -1.66533e-16
- joint Revolute 3: origin xyz=-0.0629675 0.253869 -0.0793943 rpy=-1.5708 -0 1.5708 -> xyz=0.065 0.103008 0.0125 rpy=-1.5708 -0 -1.66533e-16
- joint Revolute 4: origin xyz=-0.0629675 0.123869 -0.0793943 rpy=-1.5708 -0 1.5708 -> xyz=-0.065 0.103008 0.0125 rpy=-1.5708 -0 -1.66533e-16

File: ros2_workspace/src/simplebot_description/src/description/robot.urdf (robot description, URDF)
Before this commit: robot simplebot2, 5 links, 4 joints
Links:
- removed link base_link
- added link bottom_bracket, mass 0.426296; collision mesh filename=package://assets/bottom_bracket.stl; collision mesh filename=package://assets/frame1.stl
- link part_1: geometry collision mesh filename=package://assets/part_1__3.stl; visual mesh filename=package://assets/part_1__3.stl
- link part_1_2: geometry collision mesh filename=package://assets/part_1__3.stl; visual mesh filename=package://assets/part_1__3.stl
- link part_1_3: geometry collision mesh filename=package://assets/part_1__3.stl; visual mesh filename=package://assets/part_1__3.stl
- link part_1_4: geometry collision mesh filename=package://assets/part_1__3.stl; visual mesh filename=package://assets/part_1__3.stl
Joints:
- joint Revolute 1: origin xyz=0.143049 0.123869 -0.0793943 rpy=-1.5708 -0 1.5708 -> xyz=0.0108413 -0.0775176 -0.0147355 rpy=-1.5708 -0 -1.66533e-16; parent base_link -> bottom_bracket
- joint Revolute 2: origin xyz=0.143049 0.253869 -0.0793943 rpy=-1.5708 -0 1.5708 -> xyz=0.140841 -0.0775176 -0.0147355 rpy=-1.5708 -0 -1.66533e-16; parent base_link -> bottom_bracket
- joint Revolute 3: origin xyz=-0.0629675 0.253869 -0.0793943 rpy=1.5708 -0 1.5708 -> xyz=0.140841 0.128499 -0.0147355 rpy=-1.5708 -0 -1.66533e-16; parent base_link -> bottom_bracket
- joint Revolute 4: origin xyz=-0.0629675 0.123869 -0.0793943 rpy=1.5708 -0 1.5708 -> xyz=0.0108413 0.128499 -0.0147355 rpy=-1.5708 -0 -1.66533e-16; parent base_link -> bottom_bracket

File: ros2_workspace/src/simplebot_description/src/description/simplebot_description.urdf (robot description, URDF)
Before this commit: robot simplebot2, 5 links, 4 joints
Joints:
- joint Revolute 1: origin xyz=0.143049 0.123869 -0.0793943 rpy=-1.5708 -0 1.5708 -> xyz=-0.065 -0.103008 0.0125 rpy=-1.5708 -0 -1.66533e-16; type continuous -> revolute
- joint Revolute 2: origin xyz=0.143049 0.253869 -0.0793943 rpy=-1.5708 -0 1.5708 -> xyz=0.065 -0.103008 0.0125 rpy=-1.5708 -0 -1.66533e-16; type continuous -> revolute
- joint Revolute 3: origin xyz=-0.0629675 0.253869 -0.0793943 rpy=-1.5708 -0 1.5708 -> xyz=0.065 0.103008 0.0125 rpy=-1.5708 -0 -1.66533e-16; type continuous -> revolute
- joint Revolute 4: origin xyz=-0.0629675 0.123869 -0.0793943 rpy=-1.5708 -0 1.5708 -> xyz=-0.065 0.103008 0.0125 rpy=-1.5708 -0 -1.66533e-16; type continuous -> revolute
