Commit message: start point of urdf

File: ros2_workspace/src/roarm_ws/src/roarm_main/roarm_description/urdf/roarm_m2/roarm_m2.xacro (robot description, xacro)
@@ -5,5 +5,5 @@
 <xacro:include filename="$(find roarm_description)/urdf/roarm_m2/roarm_m2.gazebo" />
 <link name="world"></link>
-<link name="base_link">
+<link name="roarm_base_link">
   <inertial>
     <origin xyz="0.0032 0 0.04" rpy="0 0 0" />
@@ -14,5 +14,5 @@
     <origin xyz="0 0 0" rpy="0 0 0" />
     <geometry>
-      <mesh filename="file://$(find roarm_description)/meshes/roarm_m2/base_link.stl"  scale="1.0 1.0 1.0"/>
+      <mesh filename="file://$(find roarm_description)/meshes/roarm_m2/roarm_base_link.stl"  scale="1.0 1.0 1.0"/>
     </geometry>
     <material name="silver"/>
@@ -21,5 +21,5 @@
     <origin xyz="0 0 0" rpy="0 0 0" />
     <geometry>
-      <mesh filename="file://$(find roarm_description)/meshes/roarm_m2/base_link.stl"  scale="1.0 1.0 1.0"/>
+      <mesh filename="file://$(find roarm_description)/meshes/roarm_m2/roarm_base_link.stl"  scale="1.0 1.0 1.0"/>
     </geometry>
   </collision>
@@ -106,13 +106,13 @@
 </link>
 <link name="hand_tcp"></link>
-<joint name="world_to_base_link" type="fixed">
+<joint name="world_to_roarm_base_link" type="fixed">
   <origin xyz="0.0 0.0 0.0" rpy="0 0 0"/>
   <parent link="world"/>
-  <child link="base_link"/>
+  <child link="roarm_base_link"/>
   <axis xyz="0.0 0.0 1.0"/>
 </joint>
-<joint name="base_link_to_link1" type="revolute">
+<joint name="roarm_base_link_to_link1" type="revolute">
   <origin xyz="0.0100000008759151 0 0.123059270461044" rpy="0 0 0" />
-  <parent link="base_link" />
+  <parent link="roarm_base_link" />
   <child link="link1" />
   <axis xyz="0 0 1" />

File: ros2_workspace/src/simplebot_description/urdf/simplebot_description.xacro (robot description, xacro)
@@ -3,5 +3,12 @@
 <!-- Onshape https://cad.onshape.com/documents/58d69eaf54d5097cb2ee2932/w/94ca09f7b1264f3339bd84c4/e/3159eab8c0fb4f293d9f6567 -->
 <robot name="simplebot2" xmlns:xacro="http://www.ros.org/wiki/xacro">
+  <xacro:include filename="$(find simplebot_description)/urdf/wheel.xacro"/>
   <!-- Link base_link -->
+  <link name="base_footprint"/>
+  <joint name="base_joint" type="fixed">
+    <parent link="base_footprint"/>
+    <child link="base_link"/>
+    <origin xyz="0 0 0" rpy="0 0 0"/>
+  </joint>
   <link name="base_link">
     <inertial>
@@ -11,5 +18,5 @@
     </inertial>
     <!-- Part frame3 -->
-    <visual>
+    <visual name="frame3">
       <origin xyz="-0.085 2.42861e-17 -0.005" rpy="0 -0 -1.5708"/>
       <geometry>
@@ -20,12 +27,6 @@
       </material>
     </visual>
-    <collision>
-      <origin xyz="-0.085 2.42861e-17 -0.005" rpy="0 -0 -1.5708"/>
-      <geometry>
-        <mesh filename="file://$(find simplebot_description)/meshes/simplebot/frame3.stl"/>
-      </geometry>
-    </collision>
     <!-- Part side_bracket_right -->
-    <visual>
+    <visual name="side_bracket_right">
       <origin xyz="-0.085 1.04083e-17 -0.005" rpy="0 -0 -1.5708"/>
       <geometry>
@@ -36,12 +37,6 @@
       </material>
     </visual>
-    <collision>
-      <origin xyz="-0.085 1.04083e-17 -0.005" rpy="0 -0 -1.5708"/>
-      <geometry>
-        <mesh filename="file://$(find simplebot_description)/meshes/simplebot/side_bracket_right.stl"/>
-      </geometry>
-    </collision>
     <!-- Part frame2 -->
-    <visual>
+    <visual name="frame2">
       <origin xyz="-0.085 1.38778e-17 -0.005" rpy="0 -0 -1.5708"/>
       <geometry>
@@ -52,12 +47,6 @@
       </material>
     </visual>
-    <collision>
-      <origin xyz="-0.085 1.38778e-17 -0.005" rpy="0 -0 -1.5708"/>
-      <geometry>
-        <mesh filename="file://$(find simplebot_description)/meshes/simplebot/frame2.stl"/>
-      </geometry>
-    </collision>
     <!-- Part part_33 -->
-    <visual>
+    <visual name="part_33">
       <origin xyz="-0.085 2.42861e-17 -0.005" rpy="0 -0 -1.5708"/>
       <geometry>
@@ -68,12 +57,6 @@
       </material>
     </visual>
-    <collision>
-      <origin xyz="-0.085 2.42861e-17 -0.005" rpy="0 -0 -1.5708"/>
-      <geometry>
-        <mesh filename="file://$(find simplebot_description)/meshes/simplebot/part_33.stl"/>
-      </geometry>
-    </collision>
     <!-- Part motor_bracket_front_right -->
-    <visual>
+    <visual name="motor_bracket_front_right">
       <origin xyz="-0.085 2.77556e-17 -0.005" rpy="0 -0 -1.5708"/>
       <geometry>
@@ -84,30 +67,8 @@
       </material>
     </visual>
-    <collision>
+    <!-- Part motor_bracket_front_left -->
+    <visual name="motor_bracket_front_left">
       <origin xyz="-0.085 2.77556e-17 -0.005" rpy="0 -0 -1.5708"/>
       <geometry>
-        <mesh filename="file://$(find simplebot_description)/meshes/simplebot/motor_bracket_front_right.stl"/>
-      </geometry>
-    </collision>
-    <!-- Part part_1 -->
-    <visual>
-      <origin xyz="-0.085 2.42861e-17 -0.005" rpy="0 -0 -1.5708"/>
-      <geometry>
-        <mesh filename="file://$(find simplebot_description)/meshes/simplebot/part_1.stl"/>
-      </geometry>
-      <material name="part_1_material">
-        <color rgba="0.647059 0.647059 0.647059 1"/>
-      </material>
-    </visual>
-    <collision>
-      <origin xyz="-0.085 2.42861e-17 -0.005" rpy="0 -0 -1.5708"/>
-      <geometry>
-        <mesh filename="file://$(find simplebot_description)/meshes/simplebot/part_1.stl"/>
-      </geometry>
-    </collision>
-    <!-- Part motor_bracket_front_left -->
-    <visual>
-      <origin xyz="-0.085 2.77556e-17 -0.005" rpy="0 -0 -1.5708"/>
-      <geometry>
         <mesh filename="file://$(find simplebot_description)/meshes/simplebot/motor_bracket_front_left.stl"/>
       </geometry>
@@ -116,12 +77,6 @@
       </material>
     </visual>
-    <collision>
-      <origin xyz="-0.085 2.77556e-17 -0.005" rpy="0 -0 -1.5708"/>
-      <geometry>
-        <mesh filename="file://$(find simplebot_description)/meshes/simplebot/motor_bracket_front_left.stl"/>
-      </geometry>
-    </collision>
     <!-- Part frame4 -->
-    <visual>
+    <visual name="frame4">
       <origin xyz="-0.085 2.1684e-17 -0.005" rpy="0 -0 -1.5708"/>
       <geometry>
@@ -132,12 +87,6 @@
       </material>
     </visual>
-    <collision>
-      <origin xyz="-0.085 2.1684e-17 -0.005" rpy="0 -0 -1.5708"/>
-      <geometry>
-        <mesh filename="file://$(find simplebot_description)/meshes/simplebot/frame4.stl"/>
-      </geometry>
-    </collision>
     <!-- Part motor_bracket_rear_left -->
-    <visual>
+    <visual name="motor_bracket_rear_left">
       <origin xyz="-0.085 1.04083e-17 -0.005" rpy="0 -0 -1.5708"/>
       <geometry>
@@ -148,28 +97,6 @@
       </material>
     </visual>
-    <collision>
-      <origin xyz="-0.085 1.04083e-17 -0.005" rpy="0 -0 -1.5708"/>
-      <geometry>
-        <mesh filename="file://$(find simplebot_description)/meshes/simplebot/motor_bracket_rear_left.stl"/>
-      </geometry>
-    </collision>
-    <!-- Part part_1_2 -->
-    <visual>
-      <origin xyz="-0.085 3.46945e-18 -0.005" rpy="-6.16298e-33 -0 -1.5708"/>
-      <geometry>
-        <mesh filename="file://$(find simplebot_description)/meshes/simplebot/part_1__2.stl"/>
-      </geometry>
-      <material name="part_1_2_material">
-        <color rgba="0.231373 0.380392 0.705882 1"/>
-      </material>
-    </visual>
-    <collision>
-      <origin xyz="-0.085 3.46945e-18 -0.005" rpy="-6.16298e-33 -0 -1.5708"/>
-      <geometry>
-        <mesh filename="file://$(find simplebot_description)/meshes/simplebot/part_1__2.stl"/>
-      </geometry>
-    </collision>
     <!-- Part part_22 -->
-    <visual>
+    <visual name="part_22">
       <origin xyz="-0.085 2.42861e-17 -0.005" rpy="0 -0 -1.5708"/>
       <geometry>
@@ -180,12 +107,6 @@
       </material>
     </visual>
-    <collision>
-      <origin xyz="-0.085 2.42861e-17 -0.005" rpy="0 -0 -1.5708"/>
-      <geometry>
-        <mesh filename="file://$(find simplebot_description)/meshes/simplebot/part_22.stl"/>
-      </geometry>
-    </collision>
     <!-- Part motor_bracket_rear_right -->
-    <visual>
+    <visual name="motor_bracket_rear_right">
       <origin xyz="-0.085 1.04083e-17 -0.005" rpy="0 -0 -1.5708"/>
       <geometry>
@@ -196,12 +117,6 @@
       </material>
     </visual>
-    <collision>
-      <origin xyz="-0.085 1.04083e-17 -0.005" rpy="0 -0 -1.5708"/>
-      <geometry>
-        <mesh filename="file://$(find simplebot_description)/meshes/simplebot/motor_bracket_rear_right.stl"/>
-      </geometry>
-    </collision>
     <!-- Part frame1 -->
-    <visual>
+    <visual name="frame1">
       <origin xyz="-0.085 1.04083e-17 -0.005" rpy="0 -0 -1.5708"/>
       <geometry>
@@ -212,12 +127,6 @@
       </material>
     </visual>
-    <collision>
-      <origin xyz="-0.085 1.04083e-17 -0.005" rpy="0 -0 -1.5708"/>
-      <geometry>
-        <mesh filename="file://$(find simplebot_description)/meshes/simplebot/frame1.stl"/>
-      </geometry>
-    </collision>
     <!-- Part side_bracket_left -->
-    <visual>
+    <visual name="side_bracket_left">
       <origin xyz="-0.085 1.04083e-17 -0.005" rpy="0 -0 -1.5708"/>
       <geometry>
@@ -228,12 +137,6 @@
       </material>
     </visual>
-    <collision>
-      <origin xyz="-0.085 1.04083e-17 -0.005" rpy="0 -0 -1.5708"/>
-      <geometry>
-        <mesh filename="file://$(find simplebot_description)/meshes/simplebot/side_bracket_left.stl"/>
-      </geometry>
-    </collision>
     <!-- Part motor_front_right -->
-    <visual>
+    <visual name="motor_front_right">
       <origin xyz="0.0475 0 0.1625" rpy="-1.5708 -0 -1.5708"/>
       <geometry>
@@ -244,12 +147,6 @@
       </material>
     </visual>
-    <collision>
-      <origin xyz="0.0475 0 0.1625" rpy="-1.5708 -0 -1.5708"/>
-      <geometry>
-        <mesh filename="file://$(find simplebot_description)/meshes/simplebot/motor_front_right.stl"/>
-      </geometry>
-    </collision>
     <!-- Part motor_rear_left -->
-    <visual>
+    <visual name="motor_rear_left">
       <origin xyz="-0.0825 1.38778e-17 0.0325" rpy="-1.5708 -0 -1.5708"/>
       <geometry>
@@ -260,12 +157,6 @@
       </material>
     </visual>
-    <collision>
-      <origin xyz="-0.0825 1.38778e-17 0.0325" rpy="-1.5708 -0 -1.5708"/>
-      <geometry>
-        <mesh filename="file://$(find simplebot_description)/meshes/simplebot/motor_rear_left.stl"/>
-      </geometry>
-    </collision>
     <!-- Part motor_rear_right -->
-    <visual>
+    <visual name="motor_rear_right">
       <origin xyz="-0.0475 1.04083e-17 -0.0075" rpy="1.5708 -0 -1.5708"/>
       <geometry>
@@ -276,12 +167,6 @@
       </material>
     </visual>
-    <collision>
-      <origin xyz="-0.0475 1.04083e-17 -0.0075" rpy="1.5708 -0 -1.5708"/>
-      <geometry>
-        <mesh filename="file://$(find simplebot_description)/meshes/simplebot/motor_rear_right.stl"/>
-      </geometry>
-    </collision>
     <!-- Part base_link -->
-    <visual>
+    <visual name="chassis_plate">
       <origin xyz="-0.085 -6.93889e-18 -0.005" rpy="0 -2.31296e-16 -1.5708"/>
       <geometry>
@@ -292,12 +177,6 @@
       </material>
     </visual>
-    <collision>
-      <origin xyz="-0.085 -6.93889e-18 -0.005" rpy="0 -2.31296e-16 -1.5708"/>
-      <geometry>
-        <mesh filename="file://$(find simplebot_description)/meshes/simplebot/base_link.stl"/>
-      </geometry>
-    </collision>
     <!-- Part part_27 -->
-    <visual>
+    <visual name="part_27">
       <origin xyz="-0.085 1.04083e-17 -0.00744" rpy="0 -0 -1.5708"/>
       <geometry>
@@ -308,12 +187,6 @@
       </material>
     </visual>
-    <collision>
-      <origin xyz="-0.085 1.04083e-17 -0.00744" rpy="0 -0 -1.5708"/>
-      <geometry>
-        <mesh filename="file://$(find simplebot_description)/meshes/simplebot/part_27.stl"/>
-      </geometry>
-    </collision>
     <!-- Part motor_front_left -->
-    <visual>
+    <visual name="motor_front_left">
       <origin xyz="0.0825 -6.93889e-18 -0.1375" rpy="1.5708 -0 -1.5708"/>
       <geometry>
@@ -324,155 +197,57 @@
       </material>
     </visual>
-    <collision>
-      <origin xyz="0.0825 -6.93889e-18 -0.1375" rpy="1.5708 -0 -1.5708"/>
-      <geometry>
-        <mesh filename="file://$(find simplebot_description)/meshes/simplebot/motor_front_left.stl"/>
-      </geometry>
-    </collision>
   </link>
-  <!-- Link part_1 -->
-  <link name="part_1">
-    <inertial>
-      <origin xyz="0 0 0" rpy="0 0 0"/>
-      <mass value="0.2"/>
-      <inertia ixx="1e-09" ixy="0" ixz="0" iyy="1e-09" iyz="0" izz="1e-09"/>
-    </inertial>
-    <!-- Part part_1_3 -->
-    <visual>
-      <origin xyz="0 0 0.0075" rpy="1.5708 1.5708 0"/>
-      <geometry>
-        <mesh filename="file://$(find simplebot_description)/meshes/simplebot/part_1__3.stl"/>
-      </geometry>
-      <material name="part_1_3_material">
-        <color rgba="0.615686 0.811765 0.929412 1"/>
-      </material>
-    </visual>
-    <collision>
-      <origin xyz="0 0 0.0075" rpy="1.5708 1.5708 0"/>
-      <geometry>
-        <mesh filename="file://$(find simplebot_description)/meshes/simplebot/part_1__3.stl"/>
-      </geometry>
-    </collision>
-  </link>
-  <!-- Joint from base_link to part_1 -->
-  <joint name="Revolute_1" type="revolute">
-    <origin xyz="-0.065 -0.103008 0.0125" rpy="-1.5708 -0 -1.66533e-16"/>
-    <parent link="base_link"/>
-    <child link="part_1"/>
-    <axis xyz="0 0 1"/>
-    <limit effort="10" velocity="10" lower="-3.141592653589793" upper="3.141592653589793"/>
-  </joint>
-  <!-- Link part_1_2 -->
-  <link name="part_1_2">
-    <inertial>
-      <origin xyz="0 0 0" rpy="0 0 0"/>
-      <mass value="0.2"/>
-      <inertia ixx="1e-09" ixy="0" ixz="0" iyy="1e-09" iyz="0" izz="1e-09"/>
-    </inertial>
-    <!-- Part part_1_4 -->
-    <visual>
-      <origin xyz="0 0 0.0075" rpy="1.5708 1.5708 0"/>
-      <geometry>
-        <mesh filename="file://$(find simplebot_description)/meshes/simplebot/part_1__3.stl"/>
-      </geometry>
-      <material name="part_1_4_material">
-        <color rgba="0.615686 0.811765 0.929412 1"/>
-      </material>
-    </visual>
-    <collision>
-      <origin xyz="0 0 0.0075" rpy="1.5708 1.5708 0"/>
-      <geometry>
-        <mesh filename="file://$(find simplebot_description)/meshes/simplebot/part_1__3.stl"/>
-      </geometry>
-    </collision>
-  </link>
-  <!-- Joint from base_link to part_1_2 -->
-  <joint name="Revolute_2" type="revolute">
-    <origin xyz="0.065 -0.103008 0.0125" rpy="-1.5708 -0 -1.66533e-16"/>
-    <parent link="base_link"/>
-    <child link="part_1_2"/>
-    <axis xyz="0 0 1"/>
-    <limit effort="10" velocity="10" lower="-3.141592653589793" upper="3.141592653589793"/>
-  </joint>
-  <!-- Link part_1_3 -->
-  <link name="part_1_3">
-    <inertial>
-      <origin xyz="0 0 0" rpy="0 0 0"/>
-      <mass value="0.2"/>
-      <inertia ixx="1e-09" ixy="0" ixz="0" iyy="1e-09" iyz="0" izz="1e-09"/>
-    </inertial>
-    <!-- Part part_1_5 -->
-    <visual>
-      <origin xyz="0 0 -0.0075" rpy="-1.5708 -1.5708 0"/>
-      <geometry>
-        <mesh filename="file://$(find simplebot_description)/meshes/simplebot/part_1__3.stl"/>
-      </geometry>
-      <material name="part_1_5_material">
-        <color rgba="0.615686 0.811765 0.929412 1"/>
-      </material>
-    </visual>
-    <collision>
-      <origin xyz="0 0 -0.0075" rpy="-1.5708 -1.5708 0"/>
-      <geometry>
-        <mesh filename="file://$(find simplebot_description)/meshes/simplebot/part_1__3.stl"/>
-      </geometry>
-    </collision>
-  </link>
-  <!-- Joint from base_link to part_1_3 -->
-  <joint name="Revolute_3" type="revolute">
-    <origin xyz="0.065 0.103008 0.0125" rpy="-1.5708 -0 -1.66533e-16"/>
-    <parent link="base_link"/>
-    <child link="part_1_3"/>
-    <axis xyz="0 0 1"/>
-    <limit effort="10" velocity="10" lower="-3.141592653589793" upper="3.141592653589793"/>
-  </joint>
-  <!-- Link part_1_4 -->
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
File: ros2_workspace/src/simplebot_description/urdf/wheel.xacro (robot description, xacro)
@@ -4,13 +4,10 @@
     <link name="${name}">
       <inertial>
-        <origin xyz="0 0 0" rpy="0 0 0"/>
-        <mass value="0.2"/>
-        <inertia
-          ixx="4.78e-05" ixy="0" ixz="0"
-          iyy="4.78e-05" iyz="0"
-          izz="9.0e-05"/>
+        <mass value="0.08"/>
+        <origin xyz="0 0 0"/>
+        <inertia ixx="0.000045" iyy="0.000045" izz="0.00009" ixy="0" ixz="0" iyz="0"/>
       </inertial>
       <visual>
-        <origin xyz="0 0 0" rpy="0 0 0"/>
+        <origin xyz="0 0 0" rpy="-1.5708 0 0"/>
         <geometry>
           <cylinder radius="0.03" length="0.015"/>
@@ -21,16 +18,15 @@
       </visual>
       <collision>
-        <origin xyz="0 0 0" rpy="0 0 0"/>
+        <origin xyz="0 0 0" rpy="-1.5708 0 0"/>
         <geometry>
-          <cylinder radius="0.03" length="0.015"/>
+          <sphere radius="0.03"/>
         </geometry>
       </collision>
     </link>
-    <!-- Gazebo friction -->
     <gazebo reference="${name}">
-      <mu1>1.2</mu1>
-      <mu2>1.2</mu2>
-      <kp>100000</kp>
-      <kd>10</kd>
+      <mu1>0.5</mu1>
+      <mu2>0.5</mu2>
+      <kp>1000000.0</kp>
+      <kd>100.0</kd>
     </gazebo>
   </xacro:macro>
