Commit message: changes before antigravity

File: ros2_workspace/src/simplebot_description/urdf/simplebot_description.xacro (robot description, xacro)
@@ -5,10 +5,4 @@
   <xacro:include filename="$(find simplebot_description)/urdf/wheel.xacro"/>
   <!-- Link base_link -->
-  <link name="base_footprint"/>
-  <joint name="base_joint" type="fixed">
-    <parent link="base_footprint"/>
-    <child link="base_link"/>
-    <origin xyz="0 0 0" rpy="0 0 0"/>
-  </joint>
   <link name="base_link">
     <inertial>
@@ -17,4 +11,14 @@
       <inertia ixx="0.00184221" ixy="9.36048e-11" ixz="-1.22606e-12" iyy="0.00190478" iyz="2.8119e-08" izz="0.00332037"/>
     </inertial>
+        <!-- Part base_link -->
+    <visual name="chassis_plate">
+      <origin xyz="-0.085 -6.93889e-18 -0.005" rpy="0 -2.31296e-16 -1.5708"/>
+      <geometry>
+        <mesh filename="file://$(find simplebot_description)/meshes/simplebot/base_link.stl"/>
+      </geometry>
+      <material name="base_link_material">
+        <color rgba="0.917647 0.917647 0.917647 1"/>
+      </material>
+    </visual>
     <!-- Part frame3 -->
     <visual name="frame3">
@@ -167,14 +171,4 @@
       </material>
     </visual>
-    <!-- Part base_link -->
-    <visual name="chassis_plate">
-      <origin xyz="-0.085 -6.93889e-18 -0.005" rpy="0 -2.31296e-16 -1.5708"/>
-      <geometry>
-        <mesh filename="file://$(find simplebot_description)/meshes/simplebot/base_link.stl"/>
-      </geometry>
-      <material name="base_link_material">
-        <color rgba="0.917647 0.917647 0.917647 1"/>
-      </material>
-    </visual>
     <!-- Part part_27 -->
     <visual name="part_27">
@@ -195,4 +189,13 @@
       <material name="motor_front_left_material">
         <color rgba="0.8 0.807843 0.8 1"/>
+      </material>
+    </visual>
+    <visual>
+      <origin xyz="0.111 0 -0.005" rpy="0 0 1.5708"/>
+      <geometry>
+        <mesh filename="file://$(find simplebot_description)/meshes/simplebot/rplidar_c1.stl"/>
+      </geometry>
+      <material name="rplidar_c1_material">
+        <color rgba="0.647059 0.647059 0.647059 1"/>
       </material>
     </visual>
@@ -234,8 +237,16 @@
     filename="gz-sim-diff-drive-system"
     name="gz::sim::systems::DiffDrive">
+    <!--
       <front_left_joint>joint_front_left</front_left_joint>
       <front_right_joint>joint_front_right</front_right_joint>
       <rear_left_joint>joint_rear_left</rear_left_joint>
       <rear_right_joint>joint_rear_right</rear_right_joint>
+    -->
+      <!-- LEFT wheels -->
+      <left_joint>joint_front_left</left_joint>
+      <left_joint>joint_rear_left</left_joint>
+      <!-- RIGHT wheels -->
+      <right_joint>joint_front_right</right_joint>
+      <right_joint>joint_rear_right</right_joint>
       <wheel_separation>0.206</wheel_separation>
       <wheelbase>0.13</wheelbase>
@@ -244,5 +255,5 @@
       <odom_topic>/odom</odom_topic>
       <frame_id>odom</frame_id>
-      <child_frame_id>base_footprint</child_frame_id>
+      <child_frame_id>base_link</child_frame_id>
       <min_acceleration>-10</min_acceleration>
       <max_acceleration>10</max_acceleration>

File: ros2_workspace/src/simplebot_description/urdf/wheel.xacro (robot description, xacro)
@@ -20,14 +20,18 @@
         <origin xyz="0 0 0" rpy="-1.5708 0 0"/>
         <geometry>
-          <sphere radius="0.03"/>
+          <cylinder radius="0.03" length="0.015"/>
         </geometry>
       </collision>
     </link>
     <gazebo reference="${name}">
-      <mu1>0.5</mu1>
-      <mu2>0.5</mu2>
-      <kp>1000000.0</kp>
-      <kd>100.0</kd>
-    </gazebo>
+  <surface>
+    <friction>
+      <ode>
+        <mu>1.0</mu>
+        <mu2>1.0</mu2>
+      </ode>
+    </friction>
+  </surface>
+</gazebo>
   </xacro:macro>
 </robot>

Commit message: restore point

File: ros2_workspace/src/simplebot_description/urdf/simplebot_description.xacro (robot description, xacro)
@@ -3,4 +3,10 @@
 <!-- Onshape https://cad.onshape.com/documents/58d69eaf54d5097cb2ee2932/w/94ca09f7b1264f3339bd84c4/e/3159eab8c0fb4f293d9f6567 -->
 <robot name="simplebot2" xmlns:xacro="http://www.ros.org/wiki/xacro">
+  <link name="base_footprint"/>
+  <joint name="base_footprint_joint" type="fixed">
+    <parent link="base_footprint"/>
+    <child link="base_link"/>
+    <origin xyz="0 0 0" rpy="0 0 0"/>
+  </joint>
   <xacro:include filename="$(find simplebot_description)/urdf/wheel.xacro"/>
   <!-- Link base_link -->
@@ -21,4 +27,10 @@
       </material>
     </visual>
+    <collision>
+      <origin xyz="-0.085 0 -0.005" rpy="0 0 0"/>
+      <geometry>
+        <box size="0.25 0.16 0.02"/>
+      </geometry>
+    </collision>
     <!-- Part frame3 -->
     <visual name="frame3">
@@ -261,4 +273,12 @@
       <max_velocity>10</max_velocity>
     </plugin>
+    <plugin
+      filename="gz-sim-joint-state-publisher-system"
+      name="gz::sim::systems::JointStatePublisher">
+      <topic>/encoder_data_gz</topic> <joint_name>joint_front_left</joint_name>
+      <joint_name>joint_front_right</joint_name>
+      <joint_name>joint_rear_left</joint_name>
+      <joint_name>joint_rear_right</joint_name>
+    </plugin>
   </gazebo>
 </robot>
