Commit message: added lidar

File: ros2_workspace/src/simplebot_description/urdf/gazebo.xacro (robot description, xacro)
@@ -12,3 +12,26 @@
     </joint>
   </xacro:macro>
+    <gazebo reference="lidar_link">
+  <sensor name="lidar" type="gpu_lidar">
+    <topic>scan</topic>
+    <update_rate>10</update_rate>
+    <gz_frame_id>lidar_link</gz_frame_id>
+    <lidar>
+      <scan>
+        <horizontal>
+          <samples>720</samples>
+          <resolution>1</resolution>
+          <min_angle>-3.14159</min_angle>
+          <max_angle>3.14159</max_angle>
+        </horizontal>
+      </scan>
+      <range>
+        <min>0.15</min>
+        <max>12.0</max>
+      </range>
+    </lidar>
+    <always_on>true</always_on>
+    <visualize>true</visualize>
+  </sensor>
+</gazebo>
 </robot>

File: ros2_workspace/src/simplebot_description/urdf/parts.xacro (robot description, xacro)
@@ -28,8 +28,7 @@
     <xacro:visual_part name="side_bracket_left" mesh_file="side_bracket_left"  xyz="-0.085 1.04083e-17 -0.005" rpy="0 -0 -1.5708" color="0.6 0.6 0.6 1"/>
     <xacro:visual_part name="side_bracket_right" mesh_file="side_bracket_right"  xyz="-0.085 1.04083e-17 -0.005" rpy="0 -0 -1.5708" color="0.6 0.6 0.6 1"/>
-    <xacro:visual_part name="roarm_bracket" mesh_file="roarm_bracket"  xyz="-0.085 1.04083e-17 -0.00744" rpy="0 -0 -1.5708" color="0.6 0.6 0.6 1"/>
+    <xacro:visual_part name="roarm_bracket" mesh_file="roarm_bracket"  xyz="-0.085 1.04083e-17 -0.005" rpy="0 -0 -1.5708" color="0.6 0.6 0.6 1"/>
     <xacro:visual_part name="a010_bracket" mesh_file="a010_bracket"  xyz="-0.085 2.42861e-17 -0.005" rpy="0 -0 -1.5708" color="0.6 0.6 0.6 1"/>
     <xacro:visual_part name="top_bracket" mesh_file="top_bracket"  xyz="-0.085 2.42861e-17 -0.005" rpy="0 -0 -1.5708" color="0.6 0.6 0.6 1"/>
-    <xacro:visual_part name="lidar" mesh_file="rplidar_c1" xyz="0.111 0 -0.005" rpy="0 0 1.5708" color="0.2 0.2 0.2 1"/>
   </xacro:macro>
 </robot>

File: ros2_workspace/src/simplebot_description/urdf/robots/simplebot_description.urdf.xacro (robot description, xacro)
@@ -12,9 +12,9 @@
     <parent link="base_footprint"/>
     <child link="base_link"/>
-    <origin xyz="0 0 0" rpy="0 0 0"/>
+    <origin xyz="0 0 0.0 " rpy="0 0 0"/>
   </joint>
   <link name="base_link">
     <inertial>
-      <origin xyz="-3.23026e-10 4.0693e-18 0.0211091" rpy="0 0 0"/>
+      <origin xyz="0 0 0.0" rpy="0 0 0"/>
       <mass value="0.426296"/>
       <inertia ixx="0.00184221" ixy="9.36048e-11" ixz="-1.22606e-12" iyy="0.00190478" iyz="2.8119e-08" izz="0.00332037"/>
@@ -22,8 +22,38 @@
     <xacro:base_link_visuals />
     <collision>
-      <origin xyz="-0.085 0 -0.005" rpy="0 0 0"/>
+      <!-- <origin xyz="0.111 0 0.005" rpy="0 0 0"/> -->
+      <origin xyz="0.0 0 0.0" rpy="0 0 0"/>
       <geometry><box size="0.25 0.16 0.02"/></geometry>
     </collision>
   </link>
+    <link name="lidar_link">
+    <visual>
+      <origin xyz="0.0 0.0 0.0" rpy="0 0 1.5708"/>
+      <!-- <origin xyz="0.111 0 -0.005" rpy="0 0 1.5708"/> -->
+      <geometry>
+        <mesh filename="file://$(find simplebot_description)/meshes/simplebot/rplidar_c1_fixed.stl"/>
+      </geometry>
+      <material name="lidar_material">
+        <color rgba="0.2 0.2 0.2 1"/>
+      </material>
+    </visual>
+    <collision>
+      <geometry>
+        <cylinder radius="0.04" length="0.05"/>
+      </geometry>
+    </collision>
+    <inertial>
+      <mass value="0.2"/>
+      <origin xyz="0 0 0"/>
+      <inertia ixx="0.0001" ixy="0" ixz="0"
+              iyy="0.0001" iyz="0"
+              izz="0.0001"/>
+    </inertial>
+  </link>
+  <joint name="lidar_joint" type="fixed">
+    <parent link="base_link"/>
+    <child link="lidar_link"/>
+    <origin xyz="0.0065 0 0.098" rpy="0 0 0"/>
+  </joint>
   <xacro:drive_wheel side="left"  position="front" x="0.065"  y="0.103008"  z="0.010"/>
   <xacro:drive_wheel side="right" position="front" x="0.065"  y="-0.103008" z="0.010"/>

File: ros2_workspace/src/simplebot_description/urdf/wheel.xacro (robot description, xacro)
@@ -11,5 +11,5 @@
         <origin xyz="0 0 0" rpy="-1.5708 0 0"/>
         <geometry>
-          <cylinder radius="0.03" length="0.015"/>
+          <cylinder radius="0.033" length="0.015"/>
         </geometry>
         <material name="${name}_material">
@@ -20,5 +20,5 @@
         <origin xyz="0 0 0" rpy="-1.5708 0 0"/>
         <geometry>
-          <cylinder radius="0.03" length="0.015"/>
+          <cylinder radius="0.033" length="0.015"/>
         </geometry>
       </collision>
